File: keyboard-kicad/modern-keyboard-template.kicad_pcb (KiCad board)
At the start: 2 copper layers, 308.6 x 100 mm, 144 parts, among them J1 S2B-PH-K-S_LF__SN_, U1 nice_nano

Commit message: updated keyboard
Parts:
- J1, S1, S6: moved to B.Cu
- moved S3 428.0 mm to (303.3, 87.1)
- moved S2 423.9 mm to (305.7, 49.0)
- moved S5 352.1 mm to (170.0, 125.2), turned to 180 degrees
- moved S4 221.7 mm to (60.4, 106.2)
- moved J1 203.7 mm to (43.8, 92.6), turned to -90 degrees
- moved S1 203.6 mm to (39.1, 88.8), turned to 90 degrees
- moved S6 181.4 mm to (38.9, 80.2), turned to 90 degrees
- moved MX27 55.9 mm to (267.6, 68.0)
- moved MX42 55.9 mm to (272.4, 87.1)
- moved MX43 55.9 mm to (303.3, 87.1)
- moved MX57 55.9 mm to (315.2, 106.2)
- moved MX66 55.9 mm to (296.2, 125.2)
- moved MX67 55.9 mm to (315.2, 125.2)
- moved MX20 55.9 mm to (134.2, 68.0)
- moved MX36 55.9 mm to (158.1, 87.1)
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Connections:
- MX57 pad 1: col13 -> col12
- MX67 pad 1: col13 -> col12
- U1 pad 10: col7 -> col11
- U1 pad 11: col8 -> col12
- U1 pad 12: col9 -> col13
- U1 pad 17: unconnected-(U1-P0.31-LF-Pad17) -> row4
- U1 pad 18: unconnected-(U1-P0.29-LF-Pad18) -> row3
- U1 pad 19: unconnected-(U1-P0.02-LF-Pad19) -> row2
- U1 pad 2: col1 -> row0
- U1 pad 20: unconnected-(U1-P1.15-LF-Pad20) -> col2
- U1 pad 21: unconnected-(U1-P1.13-LF-Pad21) -> col3
- U1 pad 22: unconnected-(U1-P1.11-LF-Pad22) -> col4
- U1 pad 23: unconnected-(U1-P0.10-LF-Pad23) -> col5
- U1 pad 24: unconnected-(U1-P0.09-LF-Pad24) -> col6
- U1 pad 25: unconnected-(U1-P1.01-LF-Pad25) -> col14
- U1 pad 26: unconnected-(U1-P1.02-LF-Pad26) -> col1
- U1 pad 27: unconnected-(U1-P1.07-LF-Pad27) -> row1
- U1 pad 5: col2 -> col7
- U1 pad 6: col3 -> col8
- U1 pad 7: col4 -> col9
- U1 pad 8: col5 -> col10
- U1 pad 9: col6 -> unconnected-(U1-P1.00-Pad9)
Routing:
- net col14: track 76.2 -> 343.1 mm
- net col12: track 48.9 -> 301.5 mm, vias 0 -> 1
- net col11: track 92.0 -> 283.4 mm, vias 0 -> 1
- net col10: track 92.0 -> 267.9 mm, vias 0 -> 1
- net col13: track 80.1 -> 252.9 mm, vias 0 -> 1
- net col9: track 92.0 -> 251.6 mm, vias 0 -> 1
- net col8: track 92.0 -> 235.4 mm, vias 0 -> 1
- net col7: track 67.0 -> 194.2 mm, vias 0 -> 1
- net col6: track 67.0 -> 167.9 mm, vias 0 -> 1
- net col5: track 87.0 -> 170.8 mm, vias 0 -> 1
- net row4: track 283.4 -> 352.8 mm
- net col4: track 67.0 -> 134.3 mm, vias 0 -> 1
- net GND: track 2.54 -> 62.5 mm, vias 0 -> 1
- net col3: track 67.0 -> 119.2 mm, vias 0 -> 1
- net row3: track 273.8 -> 321.6 mm
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Other:
- board size 308.6 x 100 mm -> 308.8 x 99.1 mm

Commit message: pcb larger outline
Parts:
- moved J1 4.32 mm to (48.1, 92.8)
- moved S1 3.06 mm to (41.0, 91.2)
- moved S6 2.04 mm to (40.9, 79.8)
- moved U1 0.29 mm to (56.2, 65.9)
Routing:
- net NRST: track 20.7 -> 15.9 mm
- net Batt in: track 16.1 -> 20.3 mm, vias 0 -> 1
- net 3.7V: track 3.17 -> 6.36 mm, vias 0 -> 1
- net col1: track 102.3 -> 104.4 mm
- net GND: track 62.5 -> 62.3 mm, vias 1 -> 0
Other:
- board size 308.8 x 99.1 mm -> 306.8 x 97.2 mm

Commit message: added flower image
Parts:
- added G***: LOGO, flower:flowergraphic, B.Cu at (169.8, 124.8)
- moved U1 1.55 mm to (57.8, 65.9)
- moved S1 0.65 mm to (41.6, 91.2)
- moved S6 0.65 mm to (41.5, 79.8)
Routing:
- net col1: track 104.4 -> 101.6 mm
- net row2: track 301.9 -> 299.7 mm
- net col8: track 235.6 -> 234.0 mm
- net col6: track 168.1 -> 166.6 mm
- net col12: track 301.7 -> 300.1 mm
- net col10: track 268.1 -> 266.6 mm
- net col9: track 251.8 -> 250.3 mm
- net col7: track 194.4 -> 192.9 mm
- net col11: track 283.7 -> 282.1 mm
- net col5: track 171.1 -> 169.5 mm
- net col4: track 134.6 -> 133.1 mm
- net col3: track 119.5 -> 118.0 mm
- net col14: track 343.5 -> 341.9 mm
- net col13: track 253.2 -> 251.6 mm
- net col2: track 127.6 -> 126.1 mm
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Other:
- board size 306.8 x 97.2 mm -> 304.8 x 95.2 mm
- board text added: "karen weng"

Commit message: final kicad
Parts:
- added H1: MountingHole, MountingHole:MountingHole_2.2mm_M2, F.Cu at (58.1, 43.3)
- added H2: MountingHole, MountingHole:MountingHole_2.2mm_M2, F.Cu at (324.8, 43.3)
- added H3: MountingHole, MountingHole:MountingHole_2.2mm_M2, F.Cu at (191.4, 77.6)
- added H4: MountingHole, MountingHole:MountingHole_2.2mm_M2, F.Cu at (86.6, 117.8)
- added H5: MountingHole, MountingHole:MountingHole_2.2mm_M2, F.Cu at (305.6, 117.8)
