File: keyboard-kicad/untitled.kicad_sch (KiCad schematic)
At the start: 140 parts

Commit message: updated keyboard
Connections:
- net col12: now also MX57.1, MX67.1
- net col13: no longer MX57.1, MX67.1
Other:
- moved on the sheet: D57, D67, MX57, MX67
Changed lines of the file:
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@@
 	)
 	(junction
-		(at 246.38 149.86)
-		(diameter 0)
-		(color 0 0 0 0)
-	)
-	(junction
 		(at 195.58 114.3)
 		(diameter 0)
@@
 	)
 	(junction
-		(at 246.38 127)
-		(diameter 0)
-		(color 0 0 0 0)
-	)
-	(junction
 		(at 77.47 62.23)
 		(diameter 0)
@@
 	)
 	(junction
-		(at 215.9 127)
+		(at 231.14 127)
 		(diameter 0)
 		(color 0 0 0 0)
@@
 	)
 	(junction
+		(at 215.9 127)
+		(diameter 0)
+		(color 0 0 0 0)
+	)
+	(junction
 		(at 87.63 72.39)
 		(diameter 0)
@@
 	)
 	(junction
-		(at 215.9 149.86)
+		(at 77.47 85.09)
 		(diameter 0)
 		(color 0 0 0 0)
 	)
 	(junction
-		(at 77.47 85.09)
+		(at 210.82 114.3)
 		(diameter 0)
 		(color 0 0 0 0)
 	)
 	(junction
-		(at 210.82 114.3)
+		(at 231.14 149.86)
 		(diameter 0)
 		(color 0 0 0 0)
@@
 	)
 	(junction
-		(at 241.3 72.39)
-		(diameter 0)
-		(color 0 0 0 0)
-	)
-	(junction
 		(at 180.34 93.98)
 		(diameter 0)
@@
 	)
 	(junction
+		(at 226.06 93.98)
+		(diameter 0)
+		(color 0 0 0 0)
+	)
+	(junction
 		(at 241.3 49.53)
 		(diameter 0)
@@
 	)
 	(junction
-		(at 241.3 114.3)
-		(diameter 0)
-		(color 0 0 0 0)
-	)
-	(junction
 		(at 107.95 106.68)
 		(diameter 0)
@@
 	)
 	(junction
+		(at 226.06 114.3)
+		(diameter 0)
+		(color 0 0 0 0)
+	)
+	(junction
 		(at 256.54 93.98)
 		(diameter 0)
@@
 	)
 	(junction
+		(at 215.9 149.86)
+		(diameter 0)
+		(color 0 0 0 0)
+	)
+	(junction
 		(at 149.86 72.39)
 		(diameter 0)
@@
 	(wire
 		(pts
+			(xy 215.9 149.86) (xy 231.14 149.86)
+		)
+		(stroke
+			(width 0)
+			(type default)
+		)
+	)
+	(wire
+		(pts
 			(xy 226.06 72.39) (xy 226.06 93.98)
 		)
@@
 	(wire
 		(pts
-			(xy 246.38 149.86) (xy 261.62 149.86)
+			(xy 226.06 93.98) (xy 226.06 114.3)
 		)
 		(stroke
@@
 	(wire
 		(pts
+			(xy 226.06 114.3) (xy 226.06 137.16)
+		)
+		(stroke
+			(width 0)
+			(type default)
+		)
+	)
+	(wire
+		(pts
 			(xy 57.15 38.1) (xy 57.15 49.53)
 		)
@@
 	(wire
 		(pts
-			(xy 215.9 62.23) (xy 231.14 62.23)
-		)
-		(stroke
-			(width 0)
-			(type default)
-		)
-	)
-	(wire
-		(pts
-			(xy 139.7 62.23) (xy 154.94 62.23)
+			(xy 215.9 127) (xy 231.14 127)
 		)
 		(stroke
@@
 	(wire
 		(pts
-			(xy 57.15 114.3) (xy 57.15 137.16)
+			(xy 215.9 62.23) (xy 231.14 62.23)
 		)
 		(stroke
@@
 	(wire
 		(pts
-			(xy 215.9 149.86) (xy 246.38 149.86)
+			(xy 139.7 62.23) (xy 154.94 62.23)
 		)
 		(stroke
@@
 	(wire
 		(pts
-			(xy 241.3 72.39) (xy 241.3 114.3)
+			(xy 57.15 114.3) (xy 57.15 137.16)
 		)
 		(stroke
@@
 	(wire
 		(pts
-			(xy 215.9 85.09) (xy 231.14 85.09)
+			(xy 231.14 127) (xy 261.62 127)
 		)
 		(stroke
@@
 	(wire
 		(pts
-			(xy 87.63 72.39) (xy 87.63 93.98)
+			(xy 215.9 85.09) (xy 231.14 85.09)
 		)
 		(stroke
@@
 	(wire
 		(pts
-			(xy 107.95 106.68) (xy 123.19 106.68)
+			(xy 87.63 72.39) (xy 87.63 93.98)
 		)
 		(stroke
@@
 	(wire
 		(pts
-			(xy 123.19 149.86) (xy 170.18 149.86)
+			(xy 107.95 106.68) (xy 123.19 106.68)
 		)
 		(stroke
@@
 	(wire
 		(pts
-			(xy 215.9 127) (xy 246.38 127)
+			(xy 123.19 149.86) (xy 170.18 149.86)
 		)
 		(stroke
@@
 	(wire
 		(pts
-			(xy 246.38 127) (xy 261.62 127)
+			(xy 33.02 149.86) (xy 46.99 149.86)
 		)
 		(stroke
@@
 	(wire
 		(pts
-			(xy 33.02 149.86) (xy 46.99 149.86)
+			(xy 231.14 85.09) (xy 246.38 85.09)
 		)
 		(stroke
@@
 	(wire
 		(pts
-			(xy 231.14 85.09) (xy 246.38 85.09)
+			(xy 102.87 72.39) (xy 102.87 93.98)
 		)
 		(stroke
@@
 	(wire
 		(pts
-			(xy 102.87 72.39) (xy 102.87 93.98)
+			(xy 72.39 114.3) (xy 72.39 137.16)
 		)
 		(stroke
@@
 	(wire
 		(pts
-			(xy 72.39 114.3) (xy 72.39 137.16)
+			(xy 231.14 149.86) (xy 261.62 149.86)
 		)
 		(stroke
@@
 	(wire
 		(pts
-			(xy 241.3 114.3) (xy 241.3 137.16)
-		)
-		(stroke
-			(width 0)
-			(type default)
-		)
-	)
-	(wire
-		(pts
 			(xy 102.87 93.98) (xy 102.87 114.3)
 		)
@@
 	(symbol
 		(lib_id "Device:D")
-		(at 246.38 146.05 90)
+		(at 231.14 146.05 90)
 		(unit 1)
 		(exclude_from_sim no)
@@
 		(fields_autoplaced yes)
 		(property "Reference" "D67"
-			(at 248.92 144.7799 90)
+			(at 233.68 144.7799 90)
 			(effects
 				(font
@@
 		)
 		(property "Value" "D"
-			(at 248.92 147.3199 90)
+			(at 233.68 147.3199 90)
 			(effects
 				(font
@@
 		)
 		(property "Footprint" "Diode_SMD:D_SOD-123"
-			(at 246.38 146.05 0)
+			(at 231.14 146.05 0)
 			(effects
 				(font
@@
 		)
 		(property "Datasheet" "~"
-			(at 246.38 146.05 0)
+			(at 231.14 146.05 0)
 			(effects
 				(font
@@
 		)
 		(property "Description" "Diode"
-			(at 246.38 146.05 0)
+			(at 231.14 146.05 0)
 			(effects
 				(font
@@
 		)
 		(property "Sim.Device" "D"
-			(at 246.38 146.05 0)
+			(at 231.14 146.05 0)
 			(effects
 				(font
@@
 		)
 		(property "Sim.Pins" "1=K 2=A"
-			(at 246.38 146.05 0)
+			(at 231.14 146.05 0)
 			(effects
 				(font
@@
 	(symbol
 		(lib_id "Device:D")
-		(at 246.38 123.19 90)
+		(at 231.14 123.19 90)
 		(unit 1)
 		(exclude_from_sim no)
@@
 		(fields_autoplaced yes)
 		(property "Reference" "D57"
-			(at 248.92 121.9199 90)
+			(at 233.68 121.9199 90)
 			(effects
 				(font
@@
 		)
 		(property "Value" "D"
-			(at 248.92 124.4599 90)
+			(at 233.68 124.4599 90)
 			(effects
 				(font
@@
 		)
 		(property "Footprint" "Diode_SMD:D_SOD-123"
-			(at 246.38 123.19 0)
+			(at 231.14 123.19 0)
 			(effects
 				(font
@@
 		)
 		(property "Datasheet" "~"
-			(at 246.38 123.19 0)
+			(at 231.14 123.19 0)
 			(effects
 				(font
@@
 		)
 		(property "Description" "Diode"
-			(at 246.38 123.19 0)
+			(at 231.14 123.19 0)
 			(effects
 				(font
@@
 		)
 		(property "Sim.Device" "D"
-			(at 246.38 123.19 0)
+			(at 231.14 123.19 0)
 			(effects
 				(font
@@
 		)
 		(property "Sim.Pins" "1=K 2=A"
-			(at 246.38 123.19 0)
+			(at 231.14 123.19 0)
 			(effects
 				(font
@@
 	(symbol
 		(lib_id "PCM_marbastlib-mx:MX_SW_HS_CPG151101S11")
-		(at 243.84 116.84 0)
+		(at 228.6 116.84 0)
 		(unit 1)
 		(exclude_from_sim no)
@@
 		(fields_autoplaced yes)
 		(property "Reference" "MX57"
-			(at 243.84 109.22 0)
+			(at 228.6 109.22 0)
 			(effects
 				(font
@@
 		)
 		(property "Value" "MX_SW_HS"
-			(at 243.84 111.76 0)
+			(at 228.6 111.76 0)
 			(effects
 				(font
@@
 		)
 		(property "Footprint" "PCM_marbastlib-mx:SW_MX_HS_CPG151101S11_1u"
-			(at 243.84 116.84 0)
+			(at 228.6 116.84 0)
 			(effects
 				(font
@@
 		)
 		(property "Datasheet" "~"
-			(at 243.84 116.84 0)
+			(at 228.6 116.84 0)
 			(effects
 				(font
@@
 		)
 		(property "Description" "Push button switch, normally open, two pins, 45° tilted, Kailh CPG151101S11 for Cherry MX style switches"
-			(at 243.84 116.84 0)
+			(at 228.6 116.84 0)
 			(effects
 				(font
@@
 	(symbol
 		(lib_id "PCM_marbastlib-mx:MX_SW_HS_CPG151101S11")
-		(at 243.84 139.7 0)
+		(at 228.6 139.7 0)
 		(unit 1)
 		(exclude_from_sim no)
@@
 		(fields_autoplaced yes)
 		(property "Reference" "MX67"
-			(at 243.84 132.08 0)
+			(at 228.6 132.08 0)
 			(effects
 				(font
@@
 		)
 		(property "Value" "MX_SW_HS"
-			(at 243.84 134.62 0)
+			(at 228.6 134.62 0)
 			(effects
 				(font
@@
 		)
 		(property "Footprint" "PCM_marbastlib-mx:SW_MX_HS_CPG151101S11_1u"
-			(at 243.84 139.7 0)
+			(at 228.6 139.7 0)
 			(effects
 				(font
@@
 		)
 		(property "Datasheet" "~"
-			(at 243.84 139.7 0)
+			(at 228.6 139.7 0)
 			(effects
 				(font
@@
 		)
 		(property "Description" "Push button switch, normally open, two pins, 45° tilted, Kailh CPG151101S11 for Cherry MX style switches"
-			(at 243.84 139.7 0)
+			(at 228.6 139.7 0)
 			(effects
 				(font

Commit message: final kicad
Parts:
- added H1, H2, H3, H4, H5: MountingHole, MountingHole:MountingHole_2.2mm_M2, symbol Mechanical:MountingHole
